Commit message: implementacion de carro ackerman

File: src/f112th_sim_2501_alpha/description/lidar.xacro (robot description, xacro)
@@ -15,5 +15,5 @@
                 <cylinder radius="0.05" length="0.04"/>
             </geometry>
-            <material name="red"/>
+            <material name="orange"/>
         </visual>
         <collision>
@@ -39,5 +39,5 @@
 												<!--resolution>: this number is multiplied by samples to determine the number range data points.-->
                         <resolution>1</resolution>
-							          <min_angle>-3.14</min_angle>
+						<min_angle>-3.14</min_angle>
                         <max_angle>3.14</max_angle>
                     </horizontal>
